File: PCB/LasS0/LasS0.kicad_sch (KiCad schematic)
At the start: 0 parts

Commit message: Create initial schematic
Parts:
- added C?: 4.7nF, Capacitor_SMD:C_0603_1608Metric, symbol Device:C
- added C?: 100nF, Capacitor_SMD:C_0603_1608Metric, symbol Device:C
- added C? (x3): 10nF, Capacitor_SMD:C_0603_1608Metric, symbol Device:C
- added C? (x2): 47uF, Capacitor_SMD:C_1206_3216Metric, symbol Device:C
- added C?: 33pF, Capacitor_SMD:C_0603_1608Metric, symbol Device:C
- added D? (x3): SS14, Diode_SMD:D_SMA, symbol MeineBibli:SS14
- added J1, J2, J3, J4: CiKe2PinSock, MeineBib:Cixi_Kefa_Elec_KF2EDGR-5.08-2P, symbol Connector:Conn_01x02_Female
- added J1_1, J2_1, J3_1, J4_1: CiKe2PinPlug, symbol Connector:Conn_01x02_Male
- added JP1_A: Direct, Jumper:SolderJumper-2_P1.3mm_Open_TrianglePad1.0x1.5mm, symbol Jumper:SolderJumper_2_Open
- added JP1_B: Inverted, Jumper:SolderJumper-2_P1.3mm_Open_TrianglePad1.0x1.5mm, symbol Jumper:SolderJumper_2_Open
- added JP2_A: S0+ PU, Jumper:SolderJumper-2_P1.3mm_Open_TrianglePad1.0x1.5mm, symbol Jumper:SolderJumper_2_Open
- added JP2_B: S0- GND, Jumper:SolderJumper-2_P1.3mm_Open_TrianglePad1.0x1.5mm, symbol Jumper:SolderJumper_2_Open
- added L?: 6.8uH, MeineBib:Sunltech_SLO0630H, symbol Device:L_Iron
- added Q? (x2): S8050, Package_TO_SOT_SMD:SOT-23, symbol MeineBibli:S8050_correctpins
- added R? (x3): 1.5k, Resistor_SMD:R_0603_1608Metric, symbol Device:R
- added R? (x3): 10k, Resistor_SMD:R_0603_1608Metric, symbol Device:R
- added R? (x3): 220R, Resistor_SMD:R_0603_1608Metric, symbol Device:R
- added R?: 47K, Resistor_SMD:R_0603_1608Metric, symbol Device:R
- added U?: EL817S1, Package_DIP:SMDIP-4_W9.53mm, symbol Isolator:LTV-817S
- added U?: TPS54331D, Package_SO:SOIC-8_3.9x4.9mm_P1.27mm, symbol MeineBibli:TPS54331D
Connections:
- new net: R?.1, U?.1
- new net: Q?.3 (C), U?.2
- new net: D?.2 (A), U?.3
- new net: R?.1, U?.4
- new net: C?.1, C?.1, U?.6 (COMP)
- new net: C?.2, R?.1
- new net: JP1_A.2 (B), JP1_B.2 (B), R?.2
- new net: Q?.1 (B), R?.1 (x2)
- new net: JP1_B.1 (A), Q?.3 (C), R?.2
- new net: JP2_A.1 (A), R?.2
- new net: C?.1, U?.4 (SS)
- new net: R?.1, R?.2, U?.5 (VSNS)
- new net: R?.1, R?.2
- new net: C?.1, D?.1 (K), L?.2, U?.8 (PH)
- new net: C?.2, U?.1 (BOOT)
- new net: C?.1, C?.1, D?.2 (A), L?.1, R?.1
- new net +5V: D?.1 (K), J3.2 (Pin_2), R?.1, R?.2
- new net A0: J4.1 (Pin_1)
- new net D0: J4.2 (Pin_2), JP1_A.1 (A), R?.2
- new net GND: C?.1, C?.2, C?.2, C?.2, C?.2, C?.2, D?.2 (A), J1.2 (Pin_2), J3.1 (Pin_1), JP2_B.2 (B), Q?.2 (E), Q?.2 (E), R?.2, R?.2, U?.7 (GND)
- new net S0+: J2.2 (Pin_2), JP2_A.2 (B), R?.2
- new net S0-: D?.1 (K), J2.1 (Pin_1), JP2_B.1 (A)
- new net VCC: C?.1, C?.2, J1.1 (Pin_1), R?.1, U?.2 (VIN)
- no-connect marks 0 -> 10
Other:
- note added: "Choose one between direct and inverted output"
- note added: "Enable both for pulled-up switching keep disabled for open collector S0 out"
- note added: "S0 output"
- note added: "Sensor input"
- note added: "VCC input"
