File: PCB/LasS0/LasS0.kicad_pcb (KiCad board)
At the start: 0 parts

Commit message: Start PCB, add mechanicals
Parts:
- added C1: 100nF, Capacitor_SMD:C_0603_1608Metric, F.Cu at (95.0, 72.0)
- added C2: 10nF, Capacitor_SMD:C_0603_1608Metric, F.Cu at (106.0, 58.7)
- added C3: 10nF, Capacitor_SMD:C_0603_1608Metric, F.Cu at (86.0, 79.1)
- added C4: 10nF, Capacitor_SMD:C_0603_1608Metric, F.Cu at (102.7, 62.2)
- added C5: 4.7nF, Capacitor_SMD:C_0603_1608Metric, F.Cu at (78.4, 86.3)
- added C6: 33pF, Capacitor_SMD:C_0603_1608Metric, F.Cu at (65.9, 62.4)
- added C7: 47uF, Capacitor_SMD:C_1206_3216Metric, F.Cu at (66.7, 59.5)
- added C8: 47uF, Capacitor_SMD:C_1206_3216Metric, F.Cu at (53.1, 85.5)
- added D1: SS14, Diode_SMD:D_SMA, F.Cu at (85.7, 66.1)
- added D2: SS14, Diode_SMD:D_SMA, F.Cu at (67.5, 79.4)
- added D3: SS14, Diode_SMD:D_SMA, F.Cu at (96.7, 52.7)
- added H1: MountingHole, MeineBib:EigenesMountingHole_2.7mm_M2.5, F.Cu at (160.2, 72.0)
- added H2: MountingHole, MeineBib:EigenesMountingHole_2.7mm_M2.5, F.Cu at (136.9, 128.0)
- added J1: CiKe2PinSock, MeineBib:Cixi_Kefa_Elec_KF2EDGR-5.08-2P, F.Cu at (143.4, 137.0)
- added J2: CiKe2PinSock, MeineBib:Cixi_Kefa_Elec_KF2EDGR-5.08-2P, F.Cu at (153.6, 137.0)
- added J3: CiKe2PinSock, MeineBib:Cixi_Kefa_Elec_KF2EDGR-5.08-2P, F.Cu at (143.4, 63.0)
- added J4: CiKe2PinSock, MeineBib:Cixi_Kefa_Elec_KF2EDGR-5.08-2P, F.Cu at (153.6, 63.0)
- added JP1_A1: Direct, Jumper:SolderJumper-2_P1.3mm_Open_TrianglePad1.0x1.5mm, F.Cu at (90.8, 72.5)
- added JP1_B1: Inverted, Jumper:SolderJumper-2_P1.3mm_Open_TrianglePad1.0x1.5mm, F.Cu at (101.8, 59.2)
- added JP2_A1: S0+ PU, Jumper:SolderJumper-2_P1.3mm_Open_TrianglePad1.0x1.5mm, F.Cu at (58.1, 85.6)
- added JP2_B1: S0- GND, Jumper:SolderJumper-2_P1.3mm_Open_TrianglePad1.0x1.5mm, F.Cu at (109.8, 52.2)
- added L1: 6.8uH, MeineBib:Sunltech_SLO0630H, F.Cu at (77.4, 67.7)
- added LOGO1: Binary-6, MeineBib:Binary_6_v0.1, F.Cu at (60.5, 54.2)
- added LOGO3: OSHW, Symbol:OSHW-Symbol_6.7x6mm_SilkScreen, F.Cu at (75.3, 81.6)
- added Q1: S8050, Package_TO_SOT_SMD:SOT-23, F.Cu at (81.6, 80.3)
- added Q2: S8050, Package_TO_SOT_SMD:SOT-23, F.Cu at (65.9, 83.9)
- added R1: 47K, Resistor_SMD:R_0603_1608Metric, F.Cu at (98.7, 63.2)
- added R10: 10k, Resistor_SMD:R_0603_1608Metric, F.Cu at (109.7, 55.3)
- added R2: 10k, Resistor_SMD:R_0603_1608Metric, F.Cu at (98.7, 65.7)
- added R3: 1.5k, Resistor_SMD:R_0603_1608Metric, F.Cu at (114.0, 51.7)
- added R4: 220R, Resistor_SMD:R_0603_1608Metric, F.Cu at (81.1, 83.8)
- added R5: 1.5k, Resistor_SMD:R_0603_1608Metric, F.Cu at (98.7, 68.2)
- added R6: 10k, Resistor_SMD:R_0603_1608Metric, F.Cu at (74.4, 86.3)
- added R7: 1.5k, Resistor_SMD:R_0603_1608Metric, F.Cu at (87.6, 76.5)
- added R8: 220R, Resistor_SMD:R_0603_1608Metric, F.Cu at (83.6, 76.5)
- added R9: 220R, Resistor_SMD:R_0603_1608Metric, F.Cu at (70.3, 86.3)
- added U1: TPS54331D, Package_SO:SOIC-8_3.9x4.9mm_P1.27mm, F.Cu at (77.4, 74.9)
- added U2: EL817S1, Package_DIP:SMDIP-4_W9.53mm, F.Cu at (56.9, 80.5)
Other:
- board outline added: 29.3 x 82 mm
- copper layers 0 -> 2
- board text added: "2TE"
