File: PCB/LasS0/LasS0.kicad_pcb (KiCad board)
At the start: 2 copper layers, 29.3 x 82 mm, 38 parts, among them J1 CiKe2PinSock, J2 CiKe2PinSock, J3 CiKe2PinSock, J4 CiKe2PinSock, Q1 S8050, Q2 S8050, U1 TPS54331D, U2 EL817S1

Commit message: Update PCB:
- Switch to MOSFET input stage
- Add optional pullups/pulldowns on DO input
- Sadly make LOGO less pretty

Fabrication files are NOT updated yet, PCB version number is NOT updated yet
Parts:
- added JP2_D1: Input Pulldown, Jumper:SolderJumper-2_P1.3mm_Open_TrianglePad1.0x1.5mm, F.Cu at (145.8, 77.0)
- added JP2_U1: Input Pullup, Jumper:SolderJumper-2_P1.3mm_Open_TrianglePad1.0x1.5mm, F.Cu at (143.3, 77.0)
- added R11: 10k, Resistor_SMD:R_0603_1608Metric, F.Cu at (145.8, 73.2)
- added R12: 220R, Resistor_SMD:R_0603_1608Metric, F.Cu at (150.6, 91.5)
- Q1, Q2: value S8050 -> AO3400A
- R5: value 1.5k -> 220R
- R7: value 1.5k -> 10k
- moved R7 26.4 mm to (143.3, 73.2), turned to -90 degrees
- moved JP1_I1 8.41 mm to (153.4, 101.2)
- moved JP1_D1 8.14 mm to (151.1, 101.2)
- moved R5 6.64 mm to (151.6, 77.0), turned to -90 degrees
- moved Q2 6.01 mm to (150.6, 95.6)
- moved LOGO3 1.51 mm to (159.3, 86.9)
- moved Q1 0.11 mm to (150.6, 87.5)
- renumbered JP1_A1 to JP1_D1, JP1_B1 to JP1_I1, JP2_B1 to JP2_D2, JP2_A1 to JP2_U2
Connections:
- JP1_D1 pad 1: /D0 -> Net-(JP1_D1-Pad1)
- JP1_D1 pad 2: Net-(JP1_A1-Pad2) -> Net-(U2-Pad2)
- JP1_I1 pad 2: Net-(JP1_A1-Pad2) -> Net-(U2-Pad2)
- Q1 pad 1: Net-(Q1-Pad1) -> Net-(JP2_D1-Pad2)
- Q2 pad 3: Net-(Q2-Pad3) -> Net-(JP1_D1-Pad1)
- R5 pad 1: Net-(Q1-Pad1) -> /D0
- R5 pad 2: /D0 -> Net-(JP2_D1-Pad2)
- R7 pad 1: Net-(Q2-Pad1) -> +5V
- R7 pad 2: Net-(JP1_A1-Pad2) -> Net-(JP2_U1-Pad2)
- U2 pad 2: Net-(Q2-Pad3) -> Net-(U2-Pad2)
Routing:
- net /D0: track 29.7 -> 9.47 mm
- net Net-(JP2_D1-Pad2): track 0.00 -> 17.2 mm
- net Net-(R6-Pad2): track 6.90 -> 19.5 mm
- net Net-(U2-Pad2): track 0.00 -> 6.96 mm
- net Net-(JP1_A1-Pad2): track 5.55 -> 0.00 mm
- net Net-(Q2-Pad3): track 4.52 -> 0.00 mm
- net Net-(JP1_D1-Pad1): track 0.00 -> 4.14 mm
- net +5V: track 52.4 -> 56.0 mm
- net Net-(JP2_U1-Pad2): track 0.00 -> 2.26 mm
- net Net-(JP2_D1-Pad1): track 0.00 -> 2.26 mm
- net Net-(Q1-Pad1): track 1.95 -> 0.00 mm
- net Net-(Q2-Pad1): track 1.90 -> 3.18 mm
Other:
- board text added: "Input config Choose one: Pullup Pulldown"
