File: PCB/LasS0_AVR/LasS0.kicad_pcb (KiCad board)
At the start: 2 copper layers, 29.3 x 82 mm, 42 parts, among them J1 CiKe2PinSock, J2 CiKe2PinSock, J3 CiKe2PinSock, J4 CiKe2PinSock, Q1 AO3400A, Q2 AO3400A, U1 TPS54331D, U2 EL817S1

Commit message: [PCB] Implement AVR on PCB
Parts:
- removed the JP1_D1 at (151.1, 101.2)
- removed JP1_I1: Inverted, Jumper:SolderJumper-2_P1.3mm_Open_TrianglePad1.0x1.5mm
- removed JP2_U1: Input Pullup, Jumper:SolderJumper-2_P1.3mm_Open_TrianglePad1.0x1.5mm
- removed Q1: AO3400A, Package_TO_SOT_SMD:SOT-23
- removed R11, R6, R7: 10k, Resistor_SMD:R_0603_1608Metric
- added C10: 22pF, Capacitor_SMD:C_0603_1608Metric, F.Cu at (139.7, 77.5)
- added C11: 22pF, Capacitor_SMD:C_0603_1608Metric, F.Cu at (139.7, 74.0)
- added C9: 100nF, Capacitor_SMD:C_0603_1608Metric, F.Cu at (148.7, 71.8)
- added J10: Conn_01x01, MeineModule:PinheaderOwn, F.Cu at (135.6, 92.8)
- added J5: ICSP, MeineBib:AVR_ISP, F.Cu at (141.8, 81.4)
- added J6: Conn_01x01, MeineModule:PinheaderOwn, F.Cu at (135.6, 90.1)
- added J7: Conn_01x01, MeineModule:PinheaderOwn, F.Cu at (161.3, 76.5)
- added J8: Conn_01x01, MeineModule:PinheaderOwn, F.Cu at (161.3, 79.1)
- added J9: Conn_01x01, MeineModule:PinheaderOwn, F.Cu at (161.3, 81.6)
- added JP1_VCC1: S0+ VCC, Jumper:SolderJumper-2_P1.3mm_Open_TrianglePad1.0x1.5mm, F.Cu at (156.2, 119.0)
- added U3: ATtiny24A-SS, Package_SO:SOIC-14_3.9x8.7mm_P1.27mm, F.Cu at (151.0, 77.8)
- added Y1: 8 MHz, Crystal:Crystal_SMD_5032-2Pin_5.0x3.2mm, F.Cu at (143.3, 75.8)
- JP2_D1: value Input Pulldown -> DO PD
- R5: value 220R -> 10k
- moved LOGO3 16.7 mm to (145.5, 96.5)
- moved JP2_D1 9.60 mm to (153.4, 71.2), turned to 180 degrees
- moved R5 7.00 mm to (158.6, 76.5)
- moved Q2 5.95 mm to (152.3, 101.3)
- moved R12 5.95 mm to (152.3, 97.2)
- moved R9 1.95 mm to (154.2, 121.6)
- moved JP1_D1 0.85 mm to (161.3, 119.0)
- moved JP1_PU1 0.85 mm to (158.8, 119.0)
- renumbered JP2_D2 to JP1_D1, JP2_U2 to JP1_PU1
Connections:
- JP2_D1 pad 2: Net-(JP2_D1-Pad2) -> /D0
- Q2 pad 3: Net-(JP1_D1-Pad1) -> Net-(Q2-Pad3)
- R5 pad 1: /D0 -> Net-(JP2_D1-Pad1)
- R5 pad 2: Net-(JP2_D1-Pad2) -> GND
- U2 pad 2: Net-(U2-Pad2) -> Net-(Q2-Pad3)
Routing:
- net /RST: track 0.00 -> 17.3 mm, vias 0 -> 1
- net Net-(JP2_D1-Pad2): track 17.2 -> 0.00 mm
- net /SCK: track 0.00 -> 14.1 mm, vias 0 -> 1
- net /A0: track 0.00 -> 13.3 mm, vias 0 -> 1
- net Net-(J9-Pad1): track 0.00 -> 13.3 mm, vias 0 -> 1
- net /MISO: track 0.00 -> 13.2 mm
- net Net-(J7-Pad1): track 0.00 -> 11.0 mm, vias 0 -> 1
- net Net-(C11-Pad2): track 0.00 -> 8.64 mm
- net Net-(C10-Pad2): track 0.00 -> 8.58 mm
- net Net-(J8-Pad1): track 0.00 -> 8.02 mm, vias 0 -> 1
- net +5V: track 56.0 -> 63.7 mm
- net VCC: track 41.0 -> 48.2 mm
- net Net-(U2-Pad2): track 6.96 -> 0.00 mm
- net /D0: track 9.47 -> 15.8 mm
- net /MOSI: track 0.00 -> 6.20 mm
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Other:
- board text added: "-"
- board text added: "5V"
- board text added: "5V GND"
- board text added: "AO"
- board text added: "DO - PD_GND"
- board text added: "Logic level impulse to S0 converter Chrismettal 2021_07 github.com/Chrismettal/LasS0"
- board text added: "PA1 PA3 PA7"
- board text added: "SO+ - VCC SO+ - PU_VCC SO- - GND"
- board text removed: "+5V"
- board text removed: "38b7723"
- board text removed: "Choose one: Direct Output Inverted Output"
- board text removed: "Input config Choose one: Pullup Pulldown"
- board text removed: "Logic level impulse to S0 converter Chrismettal 2021_06 github.com/Chrismettal/LasS0"
- board text removed: "NC"
- board text removed: "Set both for pullup to VCC on S0+"
